File: manufacturing/HexGauge_V1R0/CTN.kicad_pcb (KiCad board)
At the start: 2 copper layers, 40.6 x 46.9 mm, 22 parts, among them J1 Conn_01x05_Pin, J2 Conn_01x05_Socket, Q1 2N3904, SW1 SW_DIP_x03

Commit message: Updated Board to version 3
Routing:
- net Net-(D1-A0): track 21.9 -> 21.2 mm
Changed lines of the file:
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@@
   (segment (start 135.16 101.584) (end 135.144 101.6) (width 0.8128) (layer "B.Cu") (net 12))
   (segment (start 139.782 96.52) (end 139.782 96.438) (width 0.8128) (layer "B.Cu") (net 12))
-  (segment (start 151.13 100.965) (end 153.67 98.425) (width 0.25) (layer "F.Cu") (net 14))
   (segment (start 159.299 88.502) (end 159.299 89.195) (width 0.2) (layer "F.Cu") (net 14))
   (segment (start 159.299 89.195) (end 160.02 89.916) (width 0.2) (layer "F.Cu") (net 14))
-  (segment (start 146.415 100.965) (end 151.13 100.965) (width 0.25) (layer "F.Cu") (net 14))
-  (segment (start 153.67 98.425) (end 153.67 97.155) (width 0.25) (layer "F.Cu") (net 14))
+  (segment (start 146.415 100.965) (end 149.86 100.965) (width 0.25) (layer "F.Cu") (net 14))
+  (segment (start 149.86 100.965) (end 153.67 97.155) (width 0.25) (layer "F.Cu") (net 14))
   (via (at 153.67 97.155) (size 0.8) (drill 0.4) (layers "F.Cu" "B.Cu") (net 14))
   (via (at 160.02 89.916) (size 0.8) (drill 0.4) (layers "F.Cu" "B.Cu") (net 14))
