File: manufacturing/HexGauge_V3R1/STM32F4_HexGauge_V3.kicad_pcb (KiCad board)
At the start: 4 copper layers, 49.8 x 44.2 mm, 72 parts, among them J1 USB_B_Micro, J2 Conn_ARM_SWD_TC2030-NL, J3 Micro_SD_Card, J4 Conn_01x04_Pin, Q1 Q_PMOS_GSD, SW1 SW_SPDT, SW2 SW_Omron_B3FS, U1 STM32F405RGT6, U2 TPMP2359D, U3 SN65HVD230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

Commit message: added old board
Parts:
- moved G*** 0.05 mm to (112.1, 64.3)
Routing:
- net GND: track 72.7 -> 75.4 mm, vias 38 -> 40
Changed lines of the file:
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@@
   )
   (footprint "Symbol:Gyro_Logo" (layer "F.Cu")
-    (at 112.17 64.22)
+    (at 112.141 64.262)
     (attr board_only exclude_from_pos_files exclude_from_bom)
     (fp_text reference "G***" (at 0 0) (layer "F.SilkS") hide
@@
   (segment (start 114.29 96.647) (end 113.322 96.647) (width 0.5) (layer "F.Cu") (net 2))
   (segment (start 123.9105 100.076) (end 124.476 100.076) (width 0.5) (layer "F.Cu") (net 2))
+  (segment (start 112.74 66.07) (end 112.74 65.858) (width 0.5) (layer "F.Cu") (net 2))
   (segment (start 122.174 100.076) (end 122.174 98.793) (width 0.5) (layer "F.Cu") (net 2))
   (segment (start 102.853378 91.873683) (end 103.759 92.329) (width 0.3) (layer "F.Cu") (net 2))
@@
   (segment (start 109.319992 99.314992) (end 109.319992 98.62) (width 0.5) (layer "F.Cu") (net 2))
   (segment (start 132.613 76.106528) (end 132.613 74.637) (width 0.5) (layer "F.Cu") (net 2))
+  (segment (start 113.447 65.151) (end 113.918994 65.151) (width 0.5) (layer "F.Cu") (net 2))
   (segment (start 123.9105 100.076) (end 122.174 100.076) (width 0.5) (layer "F.Cu") (net 2))
   (segment (start 109.42 70.82) (end 110.22 70.82) (width 0.3) (layer "F.Cu") (net 2))
@@
   (segment (start 107.27 77.77) (end 107.07 77.57) (width 0.5) (layer "F.Cu") (net 2))
   (segment (start 114.17 102.981) (end 114.948 103.759) (width 0.5) (layer "F.Cu") (net 2))
+  (segment (start 112.74 65.858) (end 113.447 65.151) (width 0.5) (layer "F.Cu") (net 2))
   (segment (start 106.754308 98.06) (end 105.478378 96.420317) (width 0.3) (layer "F.Cu") (net 2))
   (segment (start 114.987 103.72) (end 114.948 103.759) (width 0.5) (layer "F.Cu") (net 2))
@@
   (segment (start 125.04 64.815006) (end 125.044994 64.82) (width 0.5) (layer "F.Cu") (net 2))
   (segment (start 121.2452 77.84) (end 120.296 77.84) (width 0.5) (layer "F.Cu") (net 2))
+  (segment (start 110.64 66.07) (end 110.64 65.301) (width 0.5) (layer "F.Cu") (net 2))
   (segment (start 121.2596 77.8256) (end 121.2452 77.84) (width 0.5) (layer "F.Cu") (net 2))
   (segment (start 108.82 70.05) (end 108.82 70.22) (width 0.3) (layer "F.Cu") (net 2))
@@
   (segment (start 108.82 70.92) (end 108.82 70.05) (width 0.3) (layer "F.Cu") (net 2))
   (segment (start 110.9992 90.371041) (end 110.264 91.106241) (width 0.3) (layer "F.Cu") (net 2))
+  (segment (start 110.64 65.301) (end 110.49 65.151) (width 0.5) (layer "F.Cu") (net 2))
+  (via (at 110.49 65.151) (size 0.8) (drill 0.4) (layers "F.Cu" "B.Cu") (net 2))
   (via (at 133.7 95.2) (size 0.8) (drill 0.4) (layers "F.Cu" "B.Cu") (free) (net 2))
   (via (at 123.685016 77.965) (size 0.8) (drill 0.4) (layers "F.Cu" "B.Cu") (free) (net 2))
@@
   (via (at 125.072977 102.120012) (size 0.8) (drill 0.4) (layers "F.Cu" "B.Cu") (free) (net 2))
   (via (at 134.112 74.168) (size 0.8) (drill 0.4) (layers "F.Cu" "B.Cu") (free) (net 2))
+  (via (at 113.918994 65.151) (size 0.8) (drill 0.4) (layers "F.Cu" "B.Cu") (net 2))
   (via (at 134.8 95.2) (size 0.8) (drill 0.4) (layers "F.Cu" "B.Cu") (free) (net 2))
   (via (at 122.174 100.076) (size 0.8) (drill 0.4) (layers "F.Cu" "B.Cu") (net 2))
@@
   (segment (start 112.420006 73.620006) (end 113.620006 72.420006) (width 0.25) (layer "B.Cu") (net 26))
   (segment (start 113.41 73.11) (end 112.92 72.62) (width 0.25) (layer "F.Cu") (net 27))
-  (segment (start 105.849402 49.771111) (end 105.849402 49.773111) (width 0.25) (layer "F.Cu") (net 27))
   (segment (start 113.41 74.62) (end 113.41 73.11) (width 0.25) (layer "F.Cu") (net 27))
   (segment (start 113.4992 78.145) (end 113.4992 74.7092) (width 0.25) (layer "F.Cu") (net 27))

Commit message: Cleaned up PCB
Parts:
- moved C17 0.61 mm to (113.2, 66.7)
- moved C23 0.61 mm to (111.1, 66.7)
- moved R1 0.57 mm to (108.0, 76.4)
- moved R3 0.56 mm to (113.9, 75.2)
- moved R4 0.56 mm to (111.9, 75.2)
- moved U5 0.53 mm to (112.2, 70.1)
- moved G*** 0.51 mm to (112.1, 64.8)
- moved C24 0.44 mm to (110.2, 73.7)
- moved C18 0.06 mm to (108.8, 69.6)
Routing:
- net IMU_INT: track 16.8 -> 14.9 mm
- net GND: track 75.4 -> 76.9 mm, vias 40 -> 42
- net IMU_SDA: track 8.75 -> 7.43 mm
- net Net-(SW1-B): track 3.02 -> 2.15 mm
- net IMU_SCL: track 6.86 -> 6.33 mm
- net +3V3: track 48.1 -> 48.7 mm, vias 24 -> 25
