File: manufacturing/HexGauge_V3R1/STM32F4_HexGauge_V3.kicad_pcb (KiCad board)
At the start: 4 copper layers, 49.8 x 44.2 mm, 72 parts, among them J1 USB_B_Micro, J2 Conn_ARM_SWD_TC2030-NL, J3 Micro_SD_Card, J4 Conn_01x04_Pin, Q1 Q_PMOS_GSD, SW1 SW_Omron_B3FS, SW2 SW_SPDT, U1 STM32F405RGT6, U2 TPMP2359D, U3 SN65HVD230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

Commit message: Updated Component Selection
Better availability
Parts:
- removed J2: Conn_ARM_SWD_TC2030-NL, Connector:Tag-Connect_TC2030-IDC-NL_2x03_P1.27mm_Vertical
- added H3: ~, JLC:JLC_Tooling, F.Cu at (110.4, 63.6)
- added H4: ~, JLC:JLC_Tooling, F.Cu at (144.9, 83.8)
- added H5: ~, JLC:JLC_Tooling, F.Cu at (110.4, 104.1)
- added J5: Conn_02x05_Odd_Even, Connector_PinHeader_1.27mm:PinHeader_2x05_P1.27mm_Vertical, F.Cu at (125.1, 88.6)
- C15, C16: footprint Capacitor_SMD:C_1206_3216Metric -> Capacitor_SMD:C_1210_3225Metric
- moved F1 2.02 mm to (140.2, 91.3)
- moved G*** 1.28 mm to (113.4, 64.8)
- moved FB1 0.30 mm to (137.4, 90.3)
- moved C16 0.28 mm to (137.2, 93.8)
- moved C15 0.25 mm to (130.9, 84.6)
- moved Q1 0.17 mm to (135.4, 98.1)
Connections:
- U1 pad 11: unconnected-(U1-PC3-Pad11) -> CAN_SC
- U1 pad 36: CAN_SC -> unconnected-(U1-PB15-Pad36)
Routing:
- net SWO: track 18.7 -> 15.0 mm, vias 2 -> 1
- net SWDIO: track 11.6 -> 15.2 mm
- net SWCLK: track 16.3 -> 14.6 mm, vias 2 -> 1
- net +3V3: track 47.1 -> 45.9 mm, vias 27 -> 28
- net CAN_SC: track 16.4 -> 15.2 mm
- net NRST: track 27.1 -> 26.7 mm, vias 2 -> 1
