File: manufacturing/HexGauge_V3R1/STM32F4_HexGauge_V3.kicad_pcb (KiCad board)
At the start: 4 copper layers, 49.8 x 44.2 mm, 75 parts, among them J1 USB_B_Micro, J3 Micro_SD_Card, J4 Conn_01x04_Pin, J5 Conn_02x05_Odd_Even, Q1 Q_PMOS_GSD, SW1 SW_Panasonic_EVQPUC, SW2 SW_SPDT, U1 STM32F405RGT6, U2 TPMP2359D, U3 SN65HVD230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

Commit message: added Datasheets to components
Parts:
- L1: footprint Inductor_SMD:L_Wuerth_WE-TPC-3816 -> Inductor_SMD:L_7.3x7.3_H4.5
- SW1: value SW_Panasonic_EVQPUC -> SW_Omron_B3FS
- U6: value USBLC6-2 -> USBLC6-4
- moved L1 1.66 mm to (136.7, 84.8), turned to 90 degrees
- moved C15 1.36 mm to (130.9, 84.6)
- moved C14 0.87 mm to (132.1, 88.1), turned to 90 degrees
