File: manufacturing/HexGauge_V3R1/IMU.kicad_sch (KiCad schematic)
At the start: 18 parts, among them U1 MPU-6050, U3 SN65HVD230, U4 USBLC6-2

Commit message: Cleaned Up Schematic
Added Blockdiagram
Reannotated Symbols
Parts:
- removed R1: 1k5, Resistor_SMD:R_0402_1005Metric, symbol Device:R
- added R10: 100k, Resistor_SMD:R_0402_1005Metric, symbol Device:R
Connections:
- net CAN_RS: now also R10.2
- new net CAN_SC: R10.1
