File: manufacturing/HexGauge_V3R1/_autosave-Connectors.kicad_sch (KiCad schematic)
At the start: 14 parts, among them J1 USB_B_Micro, J3 Micro_SD_Card, J4 Conn_01x04_Pin, J5 Conn_02x05_Odd_Even, U4 USBLC6-4

Commit message: Updated Component Selection
Better availability
Parts:
- J5: footprint Connector_PinHeader_1.27mm:PinHeader_2x05_P1.27mm_Vertical_SMD -> Connector_PinHeader_1.27mm:PinHeader_2x05_P1.27mm_Vertical
Changed lines of the file:
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@@
       (effects (font (size 1.27 1.27)))
     )
-    (property "Footprint" "Connector_PinHeader_1.27mm:PinHeader_2x05_P1.27mm_Vertical_SMD" (at 137.16 63.5 0)
+    (property "Footprint" "Connector_PinHeader_1.27mm:PinHeader_2x05_P1.27mm_Vertical" (at 137.16 63.5 0)
       (effects (font (size 1.27 1.27)) hide)
     )
