File: manufacturing/HexGauge_V3R2/Connectors.kicad_sch (KiCad schematic)
At the start: 14 parts, among them J1 USB_B_Micro, J3 Micro_SD_Card, J4 Conn_01x04_Pin, J5 Conn_02x05_Odd_Even, U4 USBLC6-2

Commit message: FInalised Revision 2 Design
Parts:
- J1: footprint Connector_USB:USB_Micro-B_XKB_U254-051T-4BH83-F1S -> SamacSys_Parts:101181920002LF
Changed lines of the file:
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@@
-    (stroke (width 0) (type default))
-  )
-  (wire (pts (xy 81.28 71.12) (xy 81.28 68.58))
     (stroke (width 0) (type default))
   )
@@
   )
   (wire (pts (xy 257.81 71.12) (xy 257.81 69.85))
+    (stroke (width 0) (type default))
+  )
+  (wire (pts (xy 81.28 68.58) (xy 81.28 71.12))
     (stroke (width 0) (type default))
   )
@@
       (effects (font (size 1.27 1.27)) (justify right))
     )
-    (property "Footprint" "Connector_USB:USB_Micro-B_XKB_U254-051T-4BH83-F1S" (at 77.47 59.69 0)
-      (effects (font (size 1.27 1.27)) hide)
-    )
+    (property "Footprint" "SamacSys_Parts:101181920002LF" (at 77.47 59.69 0)
+      (effects (font (size 1.27 1.27)) hide)
+    )

Commit message: upd fields
Parts:
- C1, C6, R?: Dist (none) -> Self
- H1: Dist (none) -> Buydisplay
- J1, J3, U4: Dist (none) -> Mouser
- J4, J5: Dist (none) -> Reichelt
Changed lines of the file:
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@@
+      (effects (font (size 1.27 1.27)) hide)
+    )
+    (property "Dist" "" (at 198.12 116.84 0)
       (effects (font (size 1.27 1.27)) hide)
     )
@@
       (effects (font (size 1.27 1.27)) hide)
     )
+    (property "Dist" "" (at 198.12 120.65 0)
+      (effects (font (size 1.27 1.27)) hide)
+    )
     (instances
       (project "STM32F4_HexGauge_V3"
@@
     )
     (property "Datasheet" "~" (at 137.16 63.5 0)
+      (effects (font (size 1.27 1.27)) hide)
+    )
+    (property "Dist" "Reichelt" (at 137.16 63.5 0)
       (effects (font (size 1.27 1.27)) hide)
     )
@@
       (effects (font (size 1.27 1.27)) hide)
     )
+    (property "Dist" "Self" (at 257.81 74.93 0)
+      (effects (font (size 1.27 1.27)) hide)
+    )
     (pin "1")
     (pin "2")
@@
     )
     (property "LCSC Part #" "C397452" (at 81.28 58.42 0)
+      (effects (font (size 1.27 1.27)) hide)
+    )
+    (property "Dist" "Mouser" (at 81.28 58.42 0)
       (effects (font (size 1.27 1.27)) hide)
     )
@@
       (effects (font (size 1.27 1.27)) hide)
     )
+    (property "Dist" "Self" (at 85.09 132.08 0)
+      (effects (font (size 1.27 1.27)) hide)
+    )
     (pin "1")
     (pin "2")
@@
       (effects (font (size 1.27 1.27)) hide)
     )
+    (property "Dist" "" (at 198.12 124.46 0)
+      (effects (font (size 1.27 1.27)) hide)
+    )
     (instances
       (project "STM32F4_HexGauge_V3"
@@
     )
     (property "LCSC Part #" "" (at 39.37 118.11 0)
+      (effects (font (size 1.27 1.27)) hide)
+    )
+    (property "Dist" "Self" (at 39.37 118.11 0)
       (effects (font (size 1.27 1.27)) hide)
     )
@@
       (effects (font (size 1.27 1.27)) hide)
     )
+    (property "Dist" "Self" (at 74.93 132.08 0)
+      (effects (font (size 1.27 1.27)) hide)
+    )
     (pin "1")
     (pin "2")
@@
     )
     (property "LCSC Part #" "" (at 49.53 119.38 0)
+      (effects (font (size 1.27 1.27)) hide)
+    )
+    (property "Dist" "Buydisplay" (at 49.53 119.38 0)
       (effects (font (size 1.27 1.27)) hide)
     )
@@
       (effects (font (size 1.27 1.27)) hide)
     )
+    (property "Dist" "" (at 198.12 111.76 0)
+      (effects (font (size 1.27 1.27)) hide)
+    )
     (instances
       (project "STM32F4_HexGauge_V3"
@@
     )
     (property "LCSC Part #" "C7519" (at 55.88 59.69 0)
+      (effects (font (size 1.27 1.27)) hide)
+    )
+    (property "Dist" "Mouser" (at 55.88 59.69 0)
       (effects (font (size 1.27 1.27)) hide)
     )
@@
     )
     (property "LCSC Part #" "C428492" (at 231.14 66.04 0)
+      (effects (font (size 1.27 1.27)) hide)
+    )
+    (property "Dist" "Mouser" (at 231.14 66.04 0)
       (effects (font (size 1.27 1.27)) hide)
     )
@@
       (effects (font (size 1.27 1.27)) hide)
     )
+    (property "Dist" "Reichelt" (at 148.59 125.73 0)
+      (effects (font (size 1.27 1.27)) hide)
+    )
