File: manufacturing/HexGauge_V3R2/IMU.kicad_sch (KiCad schematic)
At the start: 18 parts, among them U1 MPU-6050, U3 SN65HVD230, U4 USBLC6-2

Commit message: upd fields
Parts:
- C1, C6, R1, R10, U1, U3: Dist (none) -> LCSC
- U4: Dist (none) -> Mouser
Changed lines of the file:
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@@
+      (effects (font (size 1.27 1.27)) hide)
+    )
+    (property "Dist" "LCSC" (at 199.39 73.66 0)
       (effects (font (size 1.27 1.27)) hide)
     )
@@
       (effects (font (size 1.27 1.27)) hide)
     )
+    (property "Dist" "LCSC" (at 189.23 73.66 0)
+      (effects (font (size 1.27 1.27)) hide)
+    )
     (pin "1")
     (pin "2")
@@
       (effects (font (size 1.27 1.27)) hide)
     )
+    (property "Dist" "LCSC" (at 133.35 73.66 0)
+      (effects (font (size 1.27 1.27)) hide)
+    )
     (pin "1")
     (pin "2")
@@
       (effects (font (size 1.27 1.27)) hide)
     )
+    (property "Dist" "LCSC" (at 76.2 53.34 0)
+      (effects (font (size 1.27 1.27)) hide)
+    )
     (pin "1")
     (pin "2")
@@
     )
     (property "LCSC Part #" "C7519" (at 220.98 69.85 0)
+      (effects (font (size 1.27 1.27)) hide)
+    )
+    (property "Dist" "Mouser" (at 220.98 69.85 0)
       (effects (font (size 1.27 1.27)) hide)
     )
@@
     )
     (property "LCSC Part #" "C12084" (at 160.02 68.58 0)
+      (effects (font (size 1.27 1.27)) hide)
+    )
+    (property "Dist" "LCSC" (at 160.02 68.58 0)
       (effects (font (size 1.27 1.27)) hide)
     )
@@
       (effects (font (size 1.27 1.27)) hide)
     )
+    (property "Dist" "LCSC" (at 133.35 66.04 0)
+      (effects (font (size 1.27 1.27)) hide)
+    )
     (pin "1")
     (pin "2")
@@
       (effects (font (size 1.27 1.27)) hide)
     )
+    (property "Dist" "LCSC" (at 194.31 69.85 0)
+      (effects (font (size 1.27 1.27)) hide)
+    )
     (pin "1")
     (pin "2")
@@
       (effects (font (size 1.27 1.27)) hide)
     )
+    (property "Dist" "LCSC" (at 93.98 91.44 0)
+      (effects (font (size 1.27 1.27)) hide)
+    )
     (pin "1")
     (pin "2")
@@
     )
     (property "LCSC Part #" "C24112" (at 63.5 77.47 0)
+      (effects (font (size 1.27 1.27)) hide)
+    )
+    (property "Dist" "LCSC" (at 63.5 77.47 0)
       (effects (font (size 1.27 1.27)) hide)
     )
@@
       (effects (font (size 1.27 1.27)) hide)
     )
+    (property "Dist" "LCSC" (at 151.13 52.07 0)
+      (effects (font (size 1.27 1.27)) hide)
+    )
     (pin "1")
     (pin "2")
@@
       (effects (font (size 1.27 1.27)) hide)
     )
+    (property "Dist" "LCSC" (at 139.7 52.07 0)
+      (effects (font (size 1.27 1.27)) hide)
+    )
     (pin "1")
     (pin "2")
@@
       (effects (font (size 1.27 1.27)) hide)
     )
+    (property "Dist" "LCSC" (at 199.39 66.04 0)
+      (effects (font (size 1.27 1.27)) hide)
+    )
     (pin "1")
     (pin "2")
@@
     )
     (property "LCSC Part #" "C25741" (at 133.35 81.28 0)
+      (effects (font (size 1.27 1.27)) hide)
+    )
+    (property "Dist" "LCSC" (at 133.35 81.28 0)
       (effects (font (size 1.27 1.27)) hide)
     )
@@
       (effects (font (size 1.27 1.27)) hide)
     )
+    (property "Dist" "LCSC" (at 189.23 66.04 0)
+      (effects (font (size 1.27 1.27)) hide)
+    )
     (pin "1")
     (pin "2")
@@
     )
     (property "LCSC Part #" "C1525" (at 147.32 81.28 0)
+      (effects (font (size 1.27 1.27)) hide)
+    )
+    (property "Dist" "LCSC" (at 147.32 81.28 0)
       (effects (font (size 1.27 1.27)) hide)
     )
@@
       (effects (font (size 1.27 1.27)) hide)
     )
+    (property "Dist" "LCSC" (at 83.82 91.44 0)
+      (effects (font (size 1.27 1.27)) hide)
+    )
     (pin "1")
     (pin "2")
@@
       (effects (font (size 1.27 1.27)) hide)
     )
+    (property "Dist" "LCSC" (at 50.8 53.34 0)
+      (effects (font (size 1.27 1.27)) hide)
+    )
